File: RPICamProject_Detailed/PwrReg3Volt.kicad_sch (KiCad schematic)
At the start: 14 parts

Commit message: PCB design updates
Changed lines of the file:
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@@
 	(wire
 		(pts
-			(xy 139.7 34.29) (xy 90.17 34.29)
+			(xy 139.7 34.29) (xy 88.9 34.29)
 		)
 		(stroke
@@
 	(wire
 		(pts
+			(xy 88.9 54.61) (xy 90.17 54.61)
+		)
+		(stroke
+			(width 0)
+			(type default)
+		)
+	)
+	(wire
+		(pts
 			(xy 191.77 34.29) (xy 205.74 34.29)
 		)
@@
 	(wire
 		(pts
-			(xy 90.17 34.29) (xy 90.17 54.61)
-		)
-		(stroke
+			(xy 88.9 34.29) (xy 88.9 54.61)
+		)
+		(stroke
