File: RPICamProject_Detailed/PwrReg5Volt.kicad_sch (KiCad schematic)
At the start: 15 parts

Commit message: PCB design updates
Changed lines of the file:
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@@
 	(wire
 		(pts
-			(xy 87.63 34.29) (xy 139.7 34.29)
+			(xy 88.9 34.29) (xy 139.7 34.29)
 		)
 		(stroke
@@
 	(wire
 		(pts
-			(xy 87.63 34.29) (xy 87.63 54.61)
+			(xy 88.9 34.29) (xy 88.9 54.61)
 		)
 		(stroke
@@
 	(wire
 		(pts
-			(xy 87.63 54.61) (xy 90.17 54.61)
+			(xy 88.9 54.61) (xy 90.17 54.61)
 		)
 		(stroke
