File: RPICamProject_Detailed/RPICamProject_Detailed.kicad_sch (KiCad schematic)
At the start: 2 parts

Commit message: PCB design updates
Other:
- sheet DC Motors renamed 3V Motors
- sheet Stepper Motors renamed 5V Motors
- sheet 3V Motors: file DCMotors.kicad_sch -> 3VMotors.kicad_sch
- sheet 5V Motors: file StepperMotors.kicad_sch -> 5VMotors.kicad_sch
Changed lines of the file:
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@@
 	(wire
 		(pts
-			(xy 152.4 85.09) (xy 127 85.09)
-		)
-		(stroke
-			(width 0)
-			(type default)
-		)
-	)
-	(wire
-		(pts
-			(xy 175.26 38.1) (xy 172.72 38.1)
+			(xy 153.67 102.87) (xy 128.27 102.87)
+		)
+		(stroke
+			(width 0)
+			(type default)
+		)
+	)
+	(wire
+		(pts
+			(xy 139.7 41.91) (xy 137.16 41.91)
 		)
 		(stroke
@@
 	(wire
 		(pts
-			(xy 149.86 80.01) (xy 152.4 80.01)
-		)
-		(stroke
-			(width 0)
-			(type default)
-		)
-	)
-	(wire
-		(pts
-			(xy 127 85.09) (xy 127 81.28)
-		)
-		(stroke
-			(width 0)
-			(type default)
-		)
-	)
-	(wire
-		(pts
-			(xy 166.37 40.64) (xy 166.37 39.37)
+			(xy 151.13 97.79) (xy 153.67 97.79)
+		)
+		(stroke
+			(width 0)
+			(type default)
+		)
+	)
+	(wire
+		(pts
+			(xy 128.27 102.87) (xy 128.27 99.06)
+		)
+		(stroke
+			(width 0)
+			(type default)
+		)
+	)
+	(wire
+		(pts
+			(xy 130.81 44.45) (xy 130.81 39.37)
 		)
 		(stroke
@@
 	(wire
 		(pts
-			(xy 172.72 38.1) (xy 172.72 34.29)
+			(xy 137.16 41.91) (xy 137.16 34.29)
 		)
 		(stroke
@@
 	(wire
 		(pts
-			(xy 175.26 40.64) (xy 166.37 40.64)
+			(xy 139.7 44.45) (xy 130.81 44.45)
 		)
 		(stroke
@@
 	(wire
 		(pts
-			(xy 160.02 43.18) (xy 175.26 43.18)
+			(xy 124.46 46.99) (xy 139.7 46.99)
 		)
 		(stroke
@@
 	(wire
 		(pts
-			(xy 152.4 82.55) (xy 133.35 82.55)
+			(xy 153.67 100.33) (xy 134.62 100.33)
 		)
 		(stroke
@@
 	(wire
 		(pts
-			(xy 160.02 41.91) (xy 160.02 43.18)
+			(xy 124.46 41.91) (xy 124.46 46.99)
 		)
 		(stroke
@@
 	(wire
 		(pts
-			(xy 133.35 82.55) (xy 133.35 77.47)
+			(xy 134.62 100.33) (xy 134.62 95.25)
 		)
 		(stroke
@@
 			(width 0)
 			(type default)
-		)
-	)
-	(global_label "RPI GPIO "
-		(shape input)
-		(at 149.86 80.01 180)
-		(fields_autoplaced yes)
-		(effects
-			(font
-				(size 1.27 1.27)
-			)
-			(justify right)
-		)
-		(property "Intersheetrefs" "${INTERSHEET_REFS}"
-			(at 137.3195 80.01 0)
-			(effects
-				(font
-					(size 1.27 1.27)
-				)
-				(justify right)
-				(hide yes)
-			)
 		)
 	)
@@
 	(symbol
 		(lib_id "power:+5V")
-		(at 166.37 39.37 0)
+		(at 130.81 39.37 0)
 		(unit 1)
 		(exclude_from_sim no)
@@
 		(fields_autoplaced yes)
 		(property "Reference" "#PWR06"
-			(at 166.37 43.18 0)
+			(at 130.81 43.18 0)
 			(effects
 				(font
@@
 		)
 		(property "Value" "+5V"
-			(at 166.37 34.29 0)
+			(at 130.81 34.29 0)
 			(effects
 				(font
@@
 		)
 		(property "Footprint" ""
-			(at 166.37 39.37 0)
+			(at 130.81 39.37 0)
 			(effects
 				(font
@@
 		)
 		(property "Datasheet" ""
-			(at 166.37 39.37 0)
+			(at 130.81 39.37 0)
 			(effects
 				(font
@@
 		)
 		(property "Description" "Power symbol creates a global label with name \"+5V\""
-			(at 166.37 39.37 0)
+			(at 130.81 39.37 0)
 			(effects
 				(font
@@
 	(symbol
 		(lib_id "power:+3.3V")
-		(at 127 81.28 0)
+		(at 128.27 99.06 0)
 		(unit 1)
 		(exclude_from_sim no)
@@
 		(fields_autoplaced yes)
 		(property "Reference" "#PWR011"
-			(at 127 85.09 0)
+			(at 128.27 102.87 0)
 			(effects
 				(font
@@
 		)
 		(property "Value" "+3V"
-			(at 127 76.2 0)
+			(at 128.27 93.98 0)
 			(effects
 				(font
@@
 		)
 		(property "Footprint" ""
-			(at 127 81.28 0)
+			(at 128.27 99.06 0)
 			(effects
 				(font
@@
 		)
 		(property "Datasheet" ""
-			(at 127 81.28 0)
+			(at 128.27 99.06 0)
 			(effects
 				(font
@@
 		)
 		(property "Description" "Power symbol creates a global label with name \"+3.3V\""
-			(at 127 81.28 0)
+			(at 128.27 99.06 0)
 			(effects
 				(font
@@
 	(symbol
 		(lib_id "power:GND")
-		(at 133.35 77.47 180)
+		(at 134.62 95.25 180)
 		(unit 1)
 		(exclude_from_sim no)
@@
 		(fields_autoplaced yes)
 		(property "Reference" "#PWR010"
-			(at 133.35 71.12 0)
+			(at 134.62 88.9 0)
 			(effects
 				(font
@@
 		)
 		(property "Value" "GND"
-			(at 133.35 72.39 0)
+			(at 134.62 90.17 0)
 			(effects
 				(font
@@
 		)
 		(property "Footprint" ""
-			(at 133.35 77.47 0)
+			(at 134.62 95.25 0)
 			(effects
 				(font
@@
 		)
 		(property "Datasheet" ""
-			(at 133.35 77.47 0)
+			(at 134.62 95.25 0)
 			(effects
 				(font
@@
 		)
 		(property "Description" "Power symbol creates a global label with name \"GND\" , ground"
-			(at 133.35 77.47 0)
+			(at 134.62 95.25 0)
 			(effects
 				(font
@@
 	(symbol
 		(lib_id "power:+12V")
-		(at 172.72 34.29 0)
+		(at 137.16 34.29 0)
 		(unit 1)
 		(exclude_from_sim no)
@@
 		(fields_autoplaced yes)
 		(property "Reference" "#PWR07"
-			(at 172.72 38.1 0)
+			(at 137.16 38.1 0)
 			(effects
 				(font
@@
 		)
 		(property "Value" "+12V"
-			(at 172.72 29.21 0)
+			(at 137.16 29.21 0)
 			(effects
 				(font
@@
 		)
 		(property "Footprint" ""
-			(at 172.72 34.29 0)
+			(at 137.16 34.29 0)
 			(effects
 				(font
@@
 		)
 		(property "Datasheet" ""
-			(at 172.72 34.29 0)
+			(at 137.16 34.29 0)
 			(effects
 				(font
@@
 		)
 		(property "Description" "Power symbol creates a global label with name \"+12V\""
-			(at 172.72 34.29 0)
+			(at 137.16 34.29 0)
 			(effects
 				(font
@@
 	(symbol
 		(lib_id "power:GND")
-		(at 160.02 41.91 180)
+		(at 124.46 41.91 180)
 		(unit 1)
 		(exclude_from_sim no)
@@
 		(fields_autoplaced yes)
 		(property "Reference" "#PWR08"
-			(at 160.02 35.56 0)
+			(at 124.46 35.56 0)
 			(effects
 				(font
@@
 		)
 		(property "Value" "GND"
-			(at 160.02 36.83 0)
+			(at 124.46 36.83 0)
 			(effects
 				(font
@@
 		)
 		(property "Footprint" ""
-			(at 160.02 41.91 0)
+			(at 124.46 41.91 0)
 			(effects
 				(font
@@
 		)
 		(property "Datasheet" ""
-			(at 160.02 41.91 0)
+			(at 124.46 41.91 0)
 			(effects
 				(font
@@
 		)
 		(property "Description" "Power symbol creates a global label with name \"GND\" , ground"
-			(at 160.02 41.91 0)
+			(at 124.46 41.91 0)
 			(effects
 				(font
@@
 	)
 	(sheet
-		(at 152.4 77.47)
+		(at 153.67 95.25)
 		(size 20.32 10.16)
 		(fields_autoplaced yes)
@@
 			(color 0 0 0 0.0000)
 		)
-		(property "Sheetname" "DC Motors"
-			(at 152.4 76.7584 0)
+		(property "Sheetname" "3V Motors"
+			(at 153.67 94.5384 0)
 			(effects
 				(font
@@
 			)
 		)
-		(property "Sheetfile" "DCMotors.kicad_sch"
-			(at 152.4 88.2146 0)
+		(property "Sheetfile" "3VMotors.kicad_sch"
+			(at 153.67 105.9946 0)
 			(effects
 				(font
@@
 		)
 		(property "Field2" ""
-			(at 152.4 77.47 0)
+			(at 153.67 95.25 0)
+			(effects
+				(font
+					(size 1.27 1.27)
+				)
+				(hide yes)
+			)
+		)
+		(property "Field3" ""
+			(at 153.67 95.25 0)
 			(effects
 				(font
@@
 		)
 		(pin "GND" input
-			(at 152.4 82.55 180)
+			(at 153.67 100.33 180)
 			(effects
 				(font
@@
 		)
 		(pin "RelayOnInput" input
-			(at 152.4 80.01 180)
+			(at 153.67 97.79 180)
 			(effects
 				(font
@@
 		)
 		(pin "3VoltsIn" input
-			(at 152.4 85.09 180)
+			(at 153.67 102.87 180)
 			(effects
 				(font
@@
 	)
 	(sheet
-		(at 175.26 35.56)
+		(at 139.7 39.37)
 		(size 12.7 10.16)
 		(fields_autoplaced yes)
@@
 			(color 0 0 0 0.0000)
 		)
-		(property "Sheetname" "Stepper Motors"
-			(at 175.26 34.8484 0)
+		(property "Sheetname" "5V Motors"
+			(at 139.7 38.6584 0)
 			(effects
 				(font
@@
 			)
 		)
-		(property "Sheetfile" "StepperMotors.kicad_sch"
-			(at 175.26 46.3046 0)
+		(property "Sheetfile" "5VMotors.kicad_sch"
+			(at 139.7 50.1146 0)
 			(effects
 				(font
@@
 		)
 		(pin "12V" input
-			(at 175.26 38.1 180)
+			(at 139.7 41.91 180)
 			(effects
 				(font
@@
 		)
 		(pin "5V" input
-			(at 175.26 40.64 180)
+			(at 139.7 44.45 180)
 			(effects
 				(font
@@
 		)
 		(pin "GND" input
-			(at 175.26 43.18 180)
-			(effects
-				(font
+			(at 139.7 46.99 180)
+			(effects
+				(font
