File: PCB/MitskiKiller/MitskiKillerV1_2C/MitskiKillerV1_2C.kicad_pcb (KiCad board)
At the start: 2 copper layers, 106 x 59.8 mm, 53 parts, among them J1 Conn_01x03, J2 Conn_01x03, J3 Pololu_Breakout_A4988, J4 Pololu_Breakout_A4988, J5 Conn_01x02, J6 Conn_01x03, J7 Conn_01x02, J8 Conn_01x03, K1 G5Q-1A, Q1 MMBT2222A, U1 TPS565208DDCR, U2 TPS565208DDCR

Commit message: Added pcb step files
Parts:
- removed ? (x4): , 
Routing:
- removed copper zone on F.Cu, net GND
